File: bmi270.kicad_sch (KiCad schematic)
At the start: 3 parts, among them U3 BMI270

Commit message: progress
Parts:
- C2, C3: footprint (none) -> Capacitor_SMD:C_0603_1608Metric
Connections:
- net BMI270_SPI_ENABLE: now reaches U3.12 (CSB)
- net BMI270_INT1: now reaches U3.4 (INT1)
- net BMI270_INT2: now reaches U3.9 (INT2)
Changed lines of the file:
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@@
+		)
+	)
+	(global_label "BMI270_INT2"
+		(shape output)
+		(at 91.44 66.04 0)
+		(fields_autoplaced yes)
+		(effects
+			(font
+				(size 1.27 1.27)
+			)
+			(justify left)
+		)
+		(property "Intersheetrefs" "${INTERSHEET_REFS}"
+			(at 106.4599 66.04 0)
+			(effects
+				(font
+					(size 1.27 1.27)
+				)
+				(justify left)
+				(hide yes)
+			)
 		)
 	)
@@
 		)
 	)
+	(global_label "BMI270_INT1"
+		(shape output)
+		(at 50.8 60.96 180)
+		(fields_autoplaced yes)
+		(effects
+			(font
+				(size 1.27 1.27)
+			)
+			(justify right)
+		)
+		(property "Intersheetrefs" "${INTERSHEET_REFS}"
+			(at 35.7801 60.96 0)
+			(effects
+				(font
+					(size 1.27 1.27)
+				)
+				(justify right)
+				(hide yes)
+			)
+		)
+	)
 	(global_label "SPI2_MISO"
 		(shape bidirectional)
@@
 				)
 				(justify right)
+				(hide yes)
+			)
+		)
+	)
+	(global_label "BMI270_SPI_ENABLE"
+		(shape input)
+		(at 91.44 58.42 0)
+		(fields_autoplaced yes)
+		(effects
+			(font
+				(size 1.27 1.27)
+			)
+			(justify left)
+		)
+		(property "Intersheetrefs" "${INTERSHEET_REFS}"
+			(at 113.4146 58.42 0)
+			(effects
+				(font
+					(size 1.27 1.27)
+				)
+				(justify left)
 				(hide yes)
 			)
@@
 			)
 		)
-		(property "Footprint" ""
+		(property "Footprint" "Capacitor_SMD:C_0603_1608Metric"
 			(at 116.84 80.01 0)
 			(effects
@@
 			)
 		)
-		(property "Footprint" ""
+		(property "Footprint" "Capacitor_SMD:C_0603_1608Metric"
 			(at 38.1 73.66 0)
 			(effects
