File: embassy-fc.kicad_pcb (KiCad board)
At the start: 2 copper layers, 3 parts, among them U1 BMI088, U2 STM32H753ZITx, U3 BMI270

Commit message: progress
Parts:
- added C2: 100nF, Capacitor_SMD:C_0603_1608Metric, F.Cu at (28.1, 61.3)
- added C3: 100nF, Capacitor_SMD:C_0603_1608Metric, F.Cu at (29.8, 63.2)
- moved U3 40.5 mm to (31.7, 60.5), turned to -45 degrees
Connections:
- U1 pad 1: unconnected-(U1-INT2-Pad1) -> BMI088_ACCEL_INT2
- U1 pad 12: unconnected-(U1-INT3-Pad12) -> BMI088_GYRO_INT1
- U1 pad 13: unconnected-(U1-INT4-Pad13) -> BMI088_GYRO_INT2
- U1 pad 14: unconnected-(U1-CSB1-Pad14) -> BMI088_CSB_ACCEL
- U1 pad 16: unconnected-(U1-INT1-Pad16) -> BMI088_ACCEL_INT1
- U1 pad 2: unconnected-(U1-NC-Pad2) -> GND
- U1 pad 5: unconnected-(U1-CSB2-Pad5) -> BMI088_CSB_GYRO
- U1 pad 7: unconnected-(U1-PS-Pad7) -> GND
- U2 pad 27: unconnected-(U2-PC1-Pad27) -> SPI2_MOSI
- U2 pad 28: unconnected-(U2-PC2_C-Pad28) -> SPI2_MISO
- U2 pad 69: unconnected-(U2-PB10-Pad69) -> SPI2_SCK
- U3 pad 1: unconnected-(U3-SDO-Pad1) -> SPI2_MISO
- U3 pad 13: unconnected-(U3-SCX-Pad13) -> SPI2_SCK
- U3 pad 14: unconnected-(U3-SDX-Pad14) -> SPI2_MOSI
- U3 pad 4: unconnected-(U3-INT1-Pad4) -> BMI270_INT1
- U3 pad 5: unconnected-(U3-VDDIO-Pad5) -> VDD
- U3 pad 6: unconnected-(U3-GNDIO-Pad6) -> Net-(U3-GNDIO)
- U3 pad 7: unconnected-(U3-GND-Pad7) -> GND
- U3 pad 8: unconnected-(U3-VDD-Pad8) -> VDDIO
- U3 pad 9: unconnected-(U3-INT2-Pad9) -> BMI270_INT2
Routing:
- net SPI2_MISO: track 0.00 -> 7.24 mm, vias 0 -> 2
- net SPI2_MOSI: track 0.00 -> 5.16 mm
